File: hardware/OV3660 3M Camera for Home Assistant V1.1.brd (EAGLE design)
At the start: 21 x 60 mm, 46 parts, among them Q11 AO3400, Q3 BSS138, U10 SPX3819-2V8, U15 ATH10, U16 SPX3819-1V2, U5 ESP32-S3-WROOM-1, U8 TLV75733PDBVR

Commit message: update hardware
Parts:
- removed C5: 10uF, A9G:DISCRETE_C0402
- added M1, M2, M3, M4: SCREW01-M1.2, user:THD1-M1.2
- moved D5 1.82 mm to (17.8, 51.1)
- moved R9 1.38 mm to (16.5, 43.3)
- moved Q11 1.34 mm to (17.6, 47.0)
- moved R8 1.33 mm to (17.0, 44.8)
- moved R15 0.99 mm to (3.00, 23.8)
- moved C2 0.84 mm to (14.7, 26.5), turned to 0 degrees
- moved BUZ 0.55 mm to (14.2, 51.6)
- moved U15 0.51 mm to (5.00, 49.4)
- moved R11 0.33 mm to (3.90, 52.1)
- moved R10 0.27 mm to (3.87, 50.2)
- moved C17 0.15 mm to (10.5, 50.3)
- moved C18 0.13 mm to (9.57, 50.3)
Connections:
- net CSI_2V8: no longer C5.2
- net GND: now also M1.1, M2.1, M3.1, M4.1; no longer C5.1
Routing:
- net IO41: track 27.9 -> 34.8 mm
- net M-1: track 5.94 -> 3.14 mm
- net IO45: track 23.5 -> 26.2 mm
- net +3V3: track 115.3 -> 117.3 mm
- net IO42: track 43.2 -> 44.9 mm
- net GND: track 11.5 -> 10.5 mm
- net IO38/SDA: track 55.5 -> 56.4 mm
- net N$33: track 3.71 -> 2.83 mm
Other:
- outline, holes or cut-outs redrawn
- board text added: "for HA v1.1"
- board text removed: "for Home Assistant v1.0"
