File: hardware/OV3660 3M Camera for Home Assistant V1.1.sch (EAGLE design)
At the start: 46 parts, among them Q11 AO3400, Q3 BSS138, U10 SPX3819-2V8, U15 ATH10, U16 SPX3819-1V2, U5 ESP32-S3-WROOM-1, U8 TLV75733PDBVR

Commit message: update hardware
Parts:
- removed C5: 10uF, A9G:DISCRETE_C-0402
- added M1, M2, M3, M4: SCREW01-M1.2, user:SCREW01-M1.2
Connections:
- net CSI_2V8: no longer C5.2
- net GND: now also M1.1, M2.1, M3.1, M4.1; no longer C5.1
Changed lines of the file:
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@@
 </variantdefs>
 <classes>
-<class number="0" name="default" width="0.2032" drill="0.3048">
-<clearance class="0" value="0.1524"/>
+<class number="0" name="default" width="0" drill="0.3048">
 </class>
 <class number="2" name="gnd" width="0.3048" drill="0.5588">
@@
 <part name="C6" library="A9G" deviceset="DISCRETE_C*" device="-0402" value="10uF"/>
 <part name="C2" library="A9G" deviceset="DISCRETE_C*" device="-0402" value="0.1uF"/>
-<part name="C5" library="A9G" deviceset="DISCRETE_C*" device="-0402" value="10uF"/>
 <part name="C7" library="A9G" deviceset="DISCRETE_C*" device="-0402" value="10uF"/>
 <part name="C9" library="A9G" deviceset="DISCRETE_C*" device="-0402" value="0.1uF"/>
@@
 <part name="R14" library="A9G" deviceset="DISCRETE_R*" device="-0402" value="5.1K"/>
 <part name="R15" library="A9G" deviceset="DISCRETE_R*" device="-0402" value="5.1K"/>
+<part name="M1" library="user" deviceset="SCREW01-M1.2" device=""/>
+<part name="M2" library="user" deviceset="SCREW01-M1.2" device=""/>
+<part name="M3" library="user" deviceset="SCREW01-M1.2" device=""/>
+<part name="M4" library="user" deviceset="SCREW01-M1.2" device=""/>
+<part name="GND4" library="supply1" deviceset="GND" device=""/>
+<part name="GND7" library="supply1" deviceset="GND" device=""/>
+<part name="GND8" library="supply1" deviceset="GND" device=""/>
+<part name="GND9" library="supply1" deviceset="GND" device=""/>
 </parts>
 <sheets>
@@
 <attribute name="VALUE" x="348.742" y="78.74" size="1.27" layer="96" rot="R180"/>
 </instance>
-<instance part="C5" gate="C" x="340.36" y="81.28" smashed="yes" rot="R90">
-<attribute name="NAME" x="337.566" y="83.82" size="1.27" layer="95" rot="R180"/>
-<attribute name="VALUE" x="337.312" y="80.01" size="1.27" layer="96" rot="R180"/>
-</instance>
 <instance part="C7" gate="C" x="339.09" y="53.34" smashed="yes" rot="R90">
 <attribute name="NAME" x="338.836" y="55.626" size="1.27" layer="95" rot="R180"/>
@@
 <attribute name="VALUE" x="39.37" y="154.178" size="1.27" layer="96" ratio="10" rot="R90"/>
 </instance>
+<instance part="M1" gate="G$1" x="149.86" y="121.92"/>
+<instance part="M2" gate="G$1" x="167.64" y="121.92"/>
+<instance part="M3" gate="G$1" x="187.96" y="121.92"/>
+<instance part="M4" gate="G$1" x="149.86" y="109.22"/>
+<instance part="GND4" gate="1" x="139.7" y="104.14"/>
+<instance part="GND7" gate="1" x="139.7" y="116.84"/>
+<instance part="GND8" gate="1" x="157.48" y="116.84"/>
+<instance part="GND9" gate="1" x="177.8" y="116.84"/>
 </instances>
 <busses>
@@
 <segment>
 <pinref part="GND5" gate="1" pin="GND"/>
-<wire x1="340.36" y1="72.39" x2="340.36" y2="77.47" width="0.1524" layer="91"/>
 <wire x1="350.52" y1="76.2" x2="350.52" y2="72.39" width="0.1524" layer="91"/>
 <wire x1="350.52" y1="72.39" x2="340.36" y2="72.39" width="0.1524" layer="91"/>
-<junction x="340.36" y="72.39"/>
 <pinref part="C2" gate="C" pin="1"/>
-<pinref part="C5" gate="C" pin="1"/>
 </segment>
 <segment>
@@
 <pinref part="GND1" gate="1" pin="GND"/>
 <wire x1="193.04" y1="74.93" x2="193.04" y2="72.39" width="0.1524" layer="91"/>
+</segment>
+<segment>
+<pinref part="GND4" gate="1" pin="GND"/>
+<wire x1="139.7" y1="106.68" x2="139.7" y2="109.22" width="0.1524" layer="91"/>
+<pinref part="M4" gate="G$1" pin="1"/>
+<wire x1="139.7" y1="109.22" x2="142.24" y2="109.22" width="0.1524" layer="91"/>
+</segment>
+<segment>
+<pinref part="GND7" gate="1" pin="GND"/>
+<wire x1="139.7" y1="119.38" x2="139.7" y2="121.92" width="0.1524" layer="91"/>
+<pinref part="M1" gate="G$1" pin="1"/>
+<wire x1="139.7" y1="121.92" x2="142.24" y2="121.92" width="0.1524" layer="91"/>
+</segment>
+<segment>
+<pinref part="GND8" gate="1" pin="GND"/>
+<wire x1="157.48" y1="119.38" x2="157.48" y2="121.92" width="0.1524" layer="91"/>
+<pinref part="M2" gate="G$1" pin="1"/>
+<wire x1="157.48" y1="121.92" x2="160.02" y2="121.92" width="0.1524" layer="91"/>
+</segment>
+<segment>
+<pinref part="GND9" gate="1" pin="GND"/>
+<wire x1="177.8" y1="119.38" x2="177.8" y2="121.92" width="0.1524" layer="91"/>
+<pinref part="M3" gate="G$1" pin="1"/>
+<wire x1="177.8" y1="121.92" x2="180.34" y2="121.92" width="0.1524" layer="91"/>
 </segment>
 </net>
@@
 <pinref part="U10" gate="G$1" pin="VOUT"/>
 <wire x1="336.55" y1="87.63" x2="340.36" y2="87.63" width="0.1524" layer="91"/>
-<wire x1="340.36" y1="87.63" x2="340.36" y2="85.09" width="0.1524" layer="91"/>
 <wire x1="340.36" y1="87.63" x2="350.52" y2="87.63" width="0.1524" layer="91"/>
 <wire x1="350.52" y1="87.63" x2="350.52" y2="83.82" width="0.1524" layer="91"/>
@@
 <label x="340.106" y="92.456" size="1.778" layer="95"/>
 <pinref part="C2" gate="C" pin="2"/>
-<pinref part="C5" gate="C" pin="2"/>
-</segment>
-</net>
+</segment>
+</net>
